File: KiCAD/ClassProject/Spring2022/Spring2022.sch (KiCad schematic (older format))
At the start: 1 part

Commit message: Added trace to R1
Parts:
- gave numbers to parts that had none: 1
Connections:
- wire segments 0 -> 5
Changed lines of the file:
@@
 $EndDescr
 $Comp
-L power:+1V0 #PWR?
+L power:+1V0 #PWR0101
 U 1 1 623E0677
 P 2850 2450
-F 0 "#PWR?" H 2850 2300 50  0001 C CNN
+F 0 "#PWR0101" H 2850 2300 50  0001 C CNN
 F 1 "+1V0" H 2865 2623 50  0000 C CNN
 F 2 "" H 2850 2450 50  0001 C CNN
@@
 $EndComp
 $Comp
-L 74_jacob:R R?
+L 74_jacob:R R1
 U 1 1 62509AAA
 P 5300 2450
-F 0 "R?" H 5370 2496 50  0000 L CNN
+F 0 "R1" H 5370 2496 50  0000 L CNN
 F 1 "R" H 5370 2405 50  0000 L CNN
 F 2 "74_jacob:R-0.25W-THRU" V 5230 2450 50  0001 C CNN
@@
 	1    0    0    -1
 $EndComp
+Wire Wire Line
+	5300 2300 5300 1900
+Wire Wire Line
+	5300 1900 6500 1900
+Wire Wire Line
+	6500 1900 6500 2800
+Wire Wire Line
+	6500 2800 5300 2800
+Wire Wire Line
+	5300 2800 5300 2600
 $EndSCHEMATC
