File: KiCAD/ClassProject/Spring2022/Spring2022.sch (KiCad schematic (older format))
At the start: 2 parts

Commit message: Updated ESP symbol
Parts:
- R1: symbol 74_jacob:R -> Spring2022-rescue:R-74_jacob
Changed lines of the file:
@@
 $EndComp
 $Comp
-L 74_jacob:R R1
+L Spring2022-rescue:R-74_jacob R1
 U 1 1 62509AAA
 P 5300 2450

Commit message: Made Patrick lib and moved ESP Symbol to Patrick lib
Parts:
- removed IC?: ESP32-C3-MINI-1-N4, ESP32C3MINI1N4, symbol ESP32-C3-MINI-1-N4:ESP32-C3-MINI-1-N4
- removed R1: R, 74_jacob:R-0.25W-THRU, symbol Spring2022-rescue:R-74_jacob
Connections:
- wire segments 5 -> 0
Changed lines of the file:
@@
 Comment4 ""
 $EndDescr
-$Comp
-L ESP32-C3-MINI-1-N4:ESP32-C3-MINI-1-N4 IC?
-U 1 1 62506547
-P 1650 1650
-F 0 "IC?" H 2300 1915 50  0000 C CNN
-F 1 "ESP32-C3-MINI-1-N4" H 2300 1824 50  0000 C CNN
-F 2 "ESP32C3MINI1N4" H 2800 1750 50  0001 L CNN
-F 3 "https://www.mouser.com/datasheet/2/891/Espressif_ESP32_C3_MINI_1_Datasheet-2006822.pdf" H 2800 1650 50  0001 L CNN
-F 4 "SMD MODULE, ESP32-C3FN4, PCB ANT" H 2800 1550 50  0001 L CNN "Description"
-F 5 "2.55" H 2800 1450 50  0001 L CNN "Height"
-F 6 "Espressif Systems" H 2800 1350 50  0001 L CNN "Manufacturer_Name"
-F 7 "ESP32-C3-MINI-1-N4" H 2800 1250 50  0001 L CNN "Manufacturer_Part_Number"
-F 8 "356-ESP32-C3-MINI1N4" H 2800 1150 50  0001 L CNN "Mouser Part Number"
-F 9 "https://www.mouser.co.uk/ProductDetail/Espressif-Systems/ESP32-C3-MINI-1-N4?qs=stqOd1AaK7%252B%2FpH3qqyGehA%3D%3D" H 2800 1050 50  0001 L CNN "Mouser Price/Stock"
-F 10 "" H 2800 950 50  0001 L CNN "Arrow Part Number"
-F 11 "" H 2800 850 50  0001 L CNN "Arrow Price/Stock"
-	1    1650 1650
-	1    0    0    -1
-$EndComp
-$Comp
-L Spring2022-rescue:R-74_jacob R1
-U 1 1 62509AAA
-P 5300 2450
-F 0 "R1" H 5370 2496 50  0000 L CNN
-F 1 "R" H 5370 2405 50  0000 L CNN
-F 2 "74_jacob:R-0.25W-THRU" V 5230 2450 50  0001 C CNN
-F 3 "~" H 5300 2450 50  0001 C CNN
-	1    5300 2450
-	1    0    0    -1
-$EndComp
-Wire Wire Line
-	5300 2300 5300 1900
-Wire Wire Line
-	5300 1900 6500 1900
-Wire Wire Line
-	6500 1900 6500 2800
-Wire Wire Line
-	6500 2800 5300 2800
-Wire Wire Line
-	5300 2800 5300 2600
 $EndSCHEMATC

Commit message: Added LED-Bar Schematic
Other:
- note added: "ELEC 74 Spring 2022 Class Project Schematic"
Changed lines of the file:
@@
 $Descr A4 11693 8268
 encoding utf-8
-Sheet 1 1
+Sheet 1 2
 Title ""
 Date ""
@@
 Comment4 ""
 $EndDescr
+Text Notes 750  750  0    118  ~ 0
+ELEC 74 Spring 2022 Class Project Schematic
+$Sheet
+S 1950 2650 750  600
+U 625B6136
+F0 "LED Bar" 50
+F1 "led-bar.sch" 50
+F2 "LED-SDI" I R 2700 2750 50
+F3 "LED-SCLK" I R 2700 2850 50
+F4 "LED-DCLK" I R 2700 2950 50
+F5 "~LED-OE" I R 2700 3050 50
+$EndSheet
 $EndSCHEMATC
