File: KiCAD/ClassProject/Spring2022/Spring2022.sch (KiCad schematic (older format))
At the start: 5 parts, among them IC1 ESP32-C3-MINI-1-N4, U1 FUB-MINI

Commit message: Schematic Complete -> Need to finish routing
Parts:
- removed IC1: ESP32-C3-MINI-1-N4, 74_Patrick B:ESP32C3MINI1N4, symbol 74_Patrick:ESP32-C3-MINI-1-N4
Other:
- moved on the sheet: U1
