File: KiCAD/ClassProject/Spring2022/led-bar.sch (KiCad schematic (older format))
At the start: 22 parts

Commit message: Wiring LED's
Parts:
- added R? (x16): R, 74_jacob:R-0.25W-THRU, symbol 74_Jacob:R
Connections:
- net GND: now also U?.8 (GND), U?.8 (GND), U?.8 (GND), U?.8 (GND), U?.8 (GND)
- net at D?.2 (K): now also R?.2 (x16)
- new net: R?.1, R?.1, R?.1, R?.1, R?.1, R?.1, R?.1, R?.1, R?.1, R?.1, R?.1, R?.1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
