File: KiCAD/ClassProject/Spring2022/led-bar.sch (KiCad schematic (older format))
At the start: 22 parts

Commit message: Wiring LED's
Connections:
- net +3V3: now also U?.10 (~SRCLR), U?.10 (~SRCLR), U?.10 (~SRCLR), U?.10 (~SRCLR), U?.10 (~SRCLR)
- net ~LED-OE: now also U?.13 (~OE), U?.13 (~OE), U?.13 (~OE), U?.13 (~OE), U?.13 (~OE)
- net at U?.1 (QB): now also D?.1 (RA) (x2)
- net at U?.15 (QA): now also D?.3 (GA) (x2)
- net at U?.2 (QC): now also D?.4 (BA) (x2)
- net at U?.3 (QD): now also D?.3 (GA) (x2)
- net at U?.1 (QB): now also D?.4 (BA) (x2)
- net at U?.15 (QA): now also D?.1 (RA) (x2)
- net at U?.2 (QC): now also D?.3 (GA) (x2)
- net at U?.3 (QD): now also D?.1 (RA) (x2)
- net at U?.4 (QE): now also D?.4 (BA) (x2)
- net at U?.5 (QF): now also D?.3 (GA) (x2)
- net at U?.6 (QG): now also D?.1 (RA) (x2)
- net at U?.7 (QH): now also D?.4 (BA) (x2)
- net at U?.1 (QB): now also D?.3 (GA) (x2)
- net at U?.15 (QA): now also D?.4 (BA) (x2)
- net at U?.2 (QC): now also D?.1 (RA) (x2)
- net at U?.3 (QD): now also D?.4 (BA) (x2)
- net at U?.4 (QE): now also D?.3 (GA) (x2)
- net at U?.5 (QF): now also D?.1 (RA) (x2)
- net at U?.6 (QG): now also D?.4 (BA) (x2)
- net at U?.7 (QH): now also D?.3 (GA) (x2)
- net at U?.4 (QE): now also D?.1 (RA)
- net at U?.5 (QF): now also D?.4 (BA)
- net at U?.6 (QG): now also D?.3 (GA)
- net at U?.7 (QH): now also D?.1 (RA)
