File: KiCAD/ClassProject/Spring2022/led-bar.sch (KiCad schematic (older format))
At the start: 38 parts

Commit message: Setup PCB and Annotated Parts
Parts:
- gave numbers to parts that had none: 38

Commit message: LED resistors update layout
Connections:
- net +3V3: now also U3.16 (VCC), U4.16 (VCC), U5.16 (VCC), U6.16 (VCC), U7.16 (VCC)
Changed lines of the file:
@@
 U 1 1 625B91E0
 P 2700 3400
-F 0 "U2" H 2950 4000 50  0000 C CNN
-F 1 "74HC595" H 2950 3950 50  0000 C CNN
+F 0 "U2" V 2300 2850 50  0000 C CNN
+F 1 "74HC595" V 2750 3300 50  0000 C CNN
 F 2 "74_jacob:SOIC-16_4.55x10.3mm_P1.27mm" H 2700 3400 50  0001 C CNN
 F 3 "http://www.ti.com/lit/ds/symlink/sn74hc595.pdf" H 2700 3400 50  0001 C CNN
@@
 U 1 1 625BC7C5
 P 4850 3400
-F 0 "U3" H 4850 4181 50  0000 C CNN
-F 1 "74HC595" H 4850 4090 50  0000 C CNN
+F 0 "U3" V 4450 2850 50  0000 C CNN
+F 1 "74HC595" V 4900 3300 50  0000 C CNN
 F 2 "74_jacob:SOIC-16_4.55x10.3mm_P1.27mm" H 4850 3400 50  0001 C CNN
 F 3 "http://www.ti.com/lit/ds/symlink/sn74hc595.pdf" H 4850 3400 50  0001 C CNN
@@
 U 1 1 625BE1F4
 P 7100 3400
-F 0 "U4" H 7100 4181 50  0000 C CNN
-F 1 "74HC595" H 7100 4090 50  0000 C CNN
+F 0 "U4" V 6700 2850 50  0000 C CNN
+F 1 "74HC595" V 7150 3300 50  0000 C CNN
 F 2 "74_jacob:SOIC-16_4.55x10.3mm_P1.27mm" H 7100 3400 50  0001 C CNN
 F 3 "http://www.ti.com/lit/ds/symlink/sn74hc595.pdf" H 7100 3400 50  0001 C CNN
@@
 U 1 1 625C0C85
 P 9450 3400
-F 0 "U5" H 9450 4181 50  0000 C CNN
-F 1 "74HC595" H 9450 4090 50  0000 C CNN
+F 0 "U5" V 9050 2850 50  0000 C CNN
+F 1 "74HC595" V 9500 3300 50  0000 C CNN
 F 2 "74_jacob:SOIC-16_4.55x10.3mm_P1.27mm" H 9450 3400 50  0001 C CNN
 F 3 "http://www.ti.com/lit/ds/symlink/sn74hc595.pdf" H 9450 3400 50  0001 C CNN
@@
 U 1 1 625C12EE
 P 11750 3400
-F 0 "U6" H 11750 4181 50  0000 C CNN
-F 1 "74HC595" H 11750 4090 50  0000 C CNN
+F 0 "U6" V 11350 2850 50  0000 C CNN
+F 1 "74HC595" V 11800 3300 50  0000 C CNN
 F 2 "74_jacob:SOIC-16_4.55x10.3mm_P1.27mm" H 11750 3400 50  0001 C CNN
 F 3 "http://www.ti.com/lit/ds/symlink/sn74hc595.pdf" H 11750 3400 50  0001 C CNN
@@
 U 1 1 625C1A11
 P 13700 3400
-F 0 "U7" H 13700 4181 50  0000 C CNN
-F 1 "74HC595" H 13700 4090 50  0000 C CNN
+F 0 "U7" V 13300 2850 50  0000 C CNN
+F 1 "74HC595" V 13750 3300 50  0000 C CNN
 F 2 "74_jacob:SOIC-16_4.55x10.3mm_P1.27mm" H 13700 3400 50  0001 C CNN
 F 3 "http://www.ti.com/lit/ds/symlink/sn74hc595.pdf" H 13700 3400 50  0001 C CNN
@@
 Wire Wire Line
 	4000 3400 4150 3400
+$Comp
+L power:+3.3V #PWR?
+U 1 1 6269EA72
+P 5550 3050
+F 0 "#PWR?" H 5550 2900 50  0001 C CNN
+F 1 "+3.3V" H 5565 3223 50  0000 C CNN
+F 2 "" H 5550 3050 50  0001 C CNN
+F 3 "" H 5550 3050 50  0001 C CNN
+	1    5550 3050
+	1    0    0    -1
+$EndComp
+$Comp
+L power:+3.3V #PWR?
+U 1 1 626B43F1
+P 7800 3050
+F 0 "#PWR?" H 7800 2900 50  0001 C CNN
+F 1 "+3.3V" H 7815 3223 50  0000 C CNN
+F 2 "" H 7800 3050 50  0001 C CNN
+F 3 "" H 7800 3050 50  0001 C CNN
+	1    7800 3050
+	1    0    0    -1
+$EndComp
+$Comp
+L power:+3.3V #PWR?
+U 1 1 626C9D2B
+P 10150 3050
+F 0 "#PWR?" H 10150 2900 50  0001 C CNN
+F 1 "+3.3V" H 10165 3223 50  0000 C CNN
+F 2 "" H 10150 3050 50  0001 C CNN
+F 3 "" H 10150 3050 50  0001 C CNN
+	1    10150 3050
+	1    0    0    -1
+$EndComp
+$Comp
+L power:+3.3V #PWR?
+U 1 1 626DF589
+P 12400 3050
+F 0 "#PWR?" H 12400 2900 50  0001 C CNN
+F 1 "+3.3V" H 12415 3223 50  0000 C CNN
+F 2 "" H 12400 3050 50  0001 C CNN
+F 3 "" H 12400 3050 50  0001 C CNN
+	1    12400 3050
+	1    0    0    -1
+$EndComp
+$Comp
+L power:+3.3V #PWR?
+U 1 1 626F4D86
+P 14350 3050
+F 0 "#PWR?" H 14350 2900 50  0001 C CNN
+F 1 "+3.3V" H 14365 3223 50  0000 C CNN
+F 2 "" H 14350 3050 50  0001 C CNN
+F 3 "" H 14350 3050 50  0001 C CNN
+	1    14350 3050
+	1    0    0    -1
+$EndComp
+Wire Wire Line
+	5450 3400 5550 3400
+Wire Wire Line
+	5550 3400 5550 3050
+Wire Wire Line
+	7700 3400 7800 3400
+Wire Wire Line
+	7800 3400 7800 3050
+Wire Wire Line
+	10050 3400 10150 3400
+Wire Wire Line
+	10150 3400 10150 3050
+Wire Wire Line
+	12350 3400 12400 3400
+Wire Wire Line
+	12400 3400 12400 3050
+Wire Wire Line
+	14300 3400 14350 3400
+Wire Wire Line
+	14350 3050 14350 3400
 $EndSCHEMATC

Commit message: Added most other student parts.
Connections:
- net GND: now also R1.1, R10.1, R11.1, R12.1, R13.1, R14.1, R15.1, R16.1, R2.1, R3.1, R4.1, R5.1, R6.1, R7.1, R8.1, R9.1
Other:
- note added: "ISSUES:\n"
Changed lines of the file:
@@
 $Descr B 17000 11000
 encoding utf-8
-Sheet 2 2
+Sheet 2 6
 Title ""
 Date ""
@@
 $EndComp
 Wire Wire Line
-	1250 7600 1250 7450
-Wire Wire Line
 	2150 7300 2150 7450
 Wire Wire Line
@@
 Wire Wire Line
 	14350 3050 14350 3400
+Text Notes 800  800  0    50   ~ 0
+ISSUES:\n
+Wire Wire Line
+	1250 7450 1250 7650
 $EndSCHEMATC

Commit message: Nearly finished schematic and routing.
Connections:
- net +3V3 renamed LED-V+
Other:
- note removed: "ISSUES:\n"
