File: KiCAD/ClassProject/Spring2022/bluetooth-microchip.sch (KiCad schematic (older format))
At the start: 1 part

Commit message: Nearly finished schematic and routing.
Parts:
- gave numbers to parts that had none: 1
Changed lines of the file:
@@
 $EndDescr
 $Comp
-L 74_Kevin:IS1871SF U?
+L 74_Kevin:IS1871SF U9
 U 1 1 626797B6
 P 5850 3400
-F 0 "U?" H 6744 3446 50  0000 L CNN
+F 0 "U9" H 6744 3446 50  0000 L CNN
 F 1 "IS1871SF" H 6744 3355 50  0000 L CNN
 F 2 "74_Kevin:Bluetooth_IC_IS1871SF-202-TRAY" H 5750 2250 50  0001 C CNN
