File: KiCAD/ClassProject/Spring2022/accelerometer.sch (KiCad schematic (older format))
At the start: 1 part

Commit message: Added accelerometer connections
Connections:
- net labels added: +3.3V, GND, INT1, INT2
- wire segments 14 -> 30
Changed lines of the file:
@@
 	3500 3500 4000 3500
 Connection ~ 4000 3500
+$Comp
+L power:GND #PWR?
+U 1 1 62644A84
+P 7300 4450
+F 0 "#PWR?" H 7300 4200 50  0001 C CNN
+F 1 "GND" H 7305 4277 50  0000 C CNN
+F 2 "" H 7300 4450 50  0001 C CNN
+F 3 "" H 7300 4450 50  0001 C CNN
+	1    7300 4450
+	1    0    0    -1
+$EndComp
+Wire Wire Line
+	7300 3700 7300 3800
+Connection ~ 7300 3800
+Wire Wire Line
+	4650 3800 4450 3800
+$Comp
+L power:+3.3V #PWR?
+U 1 1 6264686E
+P 7900 2500
+F 0 "#PWR?" H 7900 2350 50  0001 C CNN
+F 1 "+3.3V" H 7915 2673 50  0000 C CNN
+F 2 "" H 7900 2500 50  0001 C CNN
+F 3 "" H 7900 2500 50  0001 C CNN
+	1    7900 2500
+	1    0    0    -1
+$EndComp
+Wire Wire Line
+	7900 3600 7900 3500
+Wire Wire Line
+	7900 2500 7900 3500
+Connection ~ 7900 3500
+Text HLabel 7400 2500 1    50   Output ~ 0
+INT1
+Text HLabel 7500 2500 1    50   Output ~ 0
+INT2
+Wire Wire Line
+	7050 3300 7400 3300
+Wire Wire Line
+	7050 3400 7500 3400
+Wire Wire Line
+	7500 3400 7500 2500
+Wire Wire Line
+	7400 2500 7400 3300
+Wire Wire Line
+	7050 3500 7900 3500
+Wire Wire Line
+	7050 3600 7900 3600
+Wire Wire Line
+	7300 3800 7300 4450
+$Comp
+L power:GND #PWR?
+U 1 1 6264EB29
+P 4450 4450
+F 0 "#PWR?" H 4450 4200 50  0001 C CNN
+F 1 "GND" H 4455 4277 50  0000 C CNN
+F 2 "" H 4450 4450 50  0001 C CNN
+F 3 "" H 4450 4450 50  0001 C CNN
+	1    4450 4450
+	1    0    0    -1
+$EndComp
+Wire Wire Line
+	4450 3800 4450 4450
+Wire Wire Line
+	4650 3700 4450 3700
+Wire Wire Line
+	4450 3700 4450 3800
+Connection ~ 4450 3800
+Wire Wire Line
+	7050 3700 7300 3700
+Wire Wire Line
+	7050 3800 7300 3800
 $EndSCHEMATC

Commit message: Wiring for accelerometer
Connections:
- wire segments 30 -> 28
Changed lines of the file:
@@
 	1    0    0    -1
 $EndComp
-Wire Wire Line
-	7900 3600 7900 3500
-Wire Wire Line
-	7900 2500 7900 3500
-Connection ~ 7900 3500
-Text HLabel 7400 2500 1    50   Output ~ 0
+Text HLabel 8400 3300 2    50   Output ~ 0
 INT1
-Text HLabel 7500 2500 1    50   Output ~ 0
+Text HLabel 8400 3400 2    50   Output ~ 0
 INT2
-Wire Wire Line
-	7050 3300 7400 3300
-Wire Wire Line
-	7050 3400 7500 3400
-Wire Wire Line
-	7500 3400 7500 2500
-Wire Wire Line
-	7400 2500 7400 3300
-Wire Wire Line
-	7050 3500 7900 3500
-Wire Wire Line
-	7050 3600 7900 3600
 Wire Wire Line
 	7300 3800 7300 4450
@@
 Wire Wire Line
 	7050 3800 7300 3800
+Wire Wire Line
+	7050 3300 8400 3300
+Wire Wire Line
+	7050 3400 8400 3400
+Wire Wire Line
+	7050 3500 7900 3500
+Wire Wire Line
+	7900 3500 7900 2500
+Wire Wire Line
+	7100 3600 7900 3600
+Wire Wire Line
+	7900 3600 7900 3500
+Connection ~ 7900 3500
 $EndSCHEMATC

Commit message: Added pull-up Resistors and Capacitors to accelerometer
Parts:
- added C?: 0.1uF, a_pontech:CAP-NON-POLAR-0603, symbol 1_pontech:PLP-000068
- added C?: 10uF, a_pontech:CAP-NON-POLAR-0603, symbol 1_pontech:PLP-000409
- added R? (x3): 100k, a_pontech:R_0603_1608Metric, symbol 1_pontech:PLP-000029
Connections:
- wire segments 28 -> 45
Changed lines of the file:
@@
 	4100 3600 4100 2500
 Wire Wire Line
-	4650 3500 4000 3500
+	4650 3500 4550 3500
 Wire Wire Line
 	4000 3500 4000 2500
@@
 	1    0    0    -1
 $EndComp
-Text HLabel 8400 3300 2    50   Output ~ 0
+Text HLabel 9000 3300 2    50   Output ~ 0
 INT1
-Text HLabel 8400 3400 2    50   Output ~ 0
+Text HLabel 9000 3400 2    50   Output ~ 0
 INT2
 Wire Wire Line
@@
 	7050 3800 7300 3800
 Wire Wire Line
-	7050 3300 8400 3300
-Wire Wire Line
-	7050 3400 8400 3400
+	7050 3300 8100 3300
+Wire Wire Line
+	7050 3400 8550 3400
 Wire Wire Line
 	7050 3500 7900 3500
 Wire Wire Line
-	7900 3500 7900 2500
-Wire Wire Line
-	7100 3600 7900 3600
+	7900 3500 7900 2700
 Wire Wire Line
 	7900 3600 7900 3500
 Connection ~ 7900 3500
+$Comp
+L 1_pontech:PLP-000029 R?
+U 1 1 62646A21
+P 4550 2850
+F 0 "R?" H 4620 2896 50  0000 L CNN
+F 1 "100k" H 4620 2805 50  0000 L CNN
+F 2 "a_pontech:R_0603_1608Metric" V 4480 2850 50  0001 C CNN
+F 3 "~" H 4550 2850 50  0001 C CNN
+F 4 "100K 0.1W 1% 0603" H 4620 2759 50  0001 L CNN "Info"
+	1    4550 2850
+	1    0    0    -1
+$EndComp
+Wire Wire Line
+	8550 3100 8550 3400
+Connection ~ 8550 3400
+Wire Wire Line
+	8550 3400 9000 3400
+Wire Wire Line
+	8100 3100 8100 3300
+Connection ~ 8100 3300
+Wire Wire Line
+	8100 3300 9000 3300
+Wire Wire Line
+	8100 2800 8100 2700
+Wire Wire Line
+	8100 2700 7900 2700
+Connection ~ 7900 2700
+Wire Wire Line
+	7900 2700 7900 2600
+Wire Wire Line
+	8550 2800 8550 2600
+Wire Wire Line
+	8550 2600 7900 2600
+Connection ~ 7900 2600
+Wire Wire Line
+	7900 2600 7900 2500
+Connection ~ 4550 3500
+Wire Wire Line
+	4550 3500 4000 3500
+$Comp
+L power:+3.3V #PWR?
+U 1 1 6264A434
+P 4550 2500
+F 0 "#PWR?" H 4550 2350 50  0001 C CNN
+F 1 "+3.3V" H 4565 2673 50  0000 C CNN
+F 2 "" H 4550 2500 50  0001 C CNN
+F 3 "" H 4550 2500 50  0001 C CNN
+	1    4550 2500
+	1    0    0    -1
+$EndComp
+Wire Wire Line
+	4550 2700 4550 2500
+Wire Wire Line
+	4550 3000 4550 3500
+$Comp
+L 1_pontech:PLP-000029 R?
+U 1 1 6264656A
+P 8550 2950
+F 0 "R?" H 8620 2996 50  0000 L CNN
+F 1 "100k" H 8620 2905 50  0000 L CNN
+F 2 "a_pontech:R_0603_1608Metric" V 8480 2950 50  0001 C CNN
+F 3 "~" H 8550 2950 50  0001 C CNN
+F 4 "100K 0.1W 1% 0603" H 8620 2859 50  0001 L CNN "Info"
+	1    8550 2950
+	1    0    0    -1
+$EndComp
+$Comp
+L 1_pontech:PLP-000029 R?
+U 1 1 626461CF
+P 8100 2950
+F 0 "R?" H 8170 2996 50  0000 L CNN
+F 1 "100k" H 8170 2905 50  0000 L CNN
+F 2 "a_pontech:R_0603_1608Metric" V 8030 2950 50  0001 C CNN
+F 3 "~" H 8100 2950 50  0001 C CNN
+F 4 "100K 0.1W 1% 0603" H 8170 2859 50  0001 L CNN "Info"
+	1    8100 2950
+	1    0    0    -1
+$EndComp
+Wire Wire Line
+	7050 3600 7900 3600
+$Comp
+L 1_pontech:PLP-000068 C?
+U 1 1 6264FAC2
+P 1950 2900
+F 0 "C?" H 2050 3000 50  0000 L CNN
+F 1 "0.1uF" H 2050 2800 50  0000 L CNN
+F 2 "a_pontech:CAP-NON-POLAR-0603" H 2050 2450 50  0001 L CNN
+F 3 "~" H 1950 2900 50  0001 C CNN
+F 4 "0.1UF 25V 10% X7R 0603" H 2065 2809 50  0001 L CNN "Info"
+	1    1950 2900
+	1    0    0    -1
+$EndComp
+$Comp
+L 1_pontech:PLP-000409 C?
+U 1 1 6264FF78
+P 2600 2900
+F 0 "C?" H 2700 3000 50  0000 L CNN
+F 1 "10uF" H 2700 2800 50  0000 L CNN
+F 2 "a_pontech:CAP-NON-POLAR-0603" H 2700 2450 50  0001 L CNN
+F 3 "~" H 2600 2900 50  0001 C CNN
+F 4 "10UF 6.3V 20% X5R 0603" H 2715 2809 50  0001 L CNN "Info"
+	1    2600 2900
+	1    0    0    -1
+$EndComp
+$Comp
+L power:+3.3V #PWR?
+U 1 1 62652D7C
+P 2600 2500
+F 0 "#PWR?" H 2600 2350 50  0001 C CNN
+F 1 "+3.3V" H 2615 2673 50  0000 C CNN
+F 2 "" H 2600 2500 50  0001 C CNN
+F 3 "" H 2600 2500 50  0001 C CNN
+	1    2600 2500
+	1    0    0    -1
+$EndComp
+$Comp
+L power:+3.3V #PWR?
+U 1 1 62653860
+P 1950 2500
+F 0 "#PWR?" H 1950 2350 50  0001 C CNN
+F 1 "+3.3V" H 1965 2673 50  0000 C CNN
+F 2 "" H 1950 2500 50  0001 C CNN
+F 3 "" H 1950 2500 50  0001 C CNN
+	1    1950 2500
+	1    0    0    -1
+$EndComp
+Wire Wire Line
+	2600 2750 2600 2500
+Wire Wire Line
+	1950 2750 1950 2500
+$Comp
+L power:GND #PWR?
+U 1 1 6265514C
+P 2600 3400
+F 0 "#PWR?" H 2600 3150 50  0001 C CNN
+F 1 "GND" H 2605 3227 50  0000 C CNN
+F 2 "" H 2600 3400 50  0001 C CNN
+F 3 "" H 2600 3400 50  0001 C CNN
+	1    2600 3400
+	1    0    0    -1
+$EndComp
+$Comp
+L power:GND #PWR?
+U 1 1 626556B5
+P 1950 3400
+F 0 "#PWR?" H 1950 3150 50  0001 C CNN
+F 1 "GND" H 1955 3227 50  0000 C CNN
+F 2 "" H 1950 3400 50  0001 C CNN
+F 3 "" H 1950 3400 50  0001 C CNN
+	1    1950 3400
+	1    0    0    -1
+$EndComp
+Wire Wire Line
+	2600 3050 2600 3400
+Wire Wire Line
+	1950 3050 1950 3400
 $EndSCHEMATC

Commit message: Nearly finished schematic and routing.
Parts:
- added R20, R21, R22, R23, R24, R25, R26: PLP-000091, a_pontech:R_0603_1608Metric, symbol 1_pontech:PLP-000091
- C4: renamed from C?; value 0.1uF -> PLP-000068
- C5: renamed from C?; value 10uF -> PLP-000409
- R27, R28, R29: renamed from R?; value 100k -> PLP-000029
- U12: renamed from U?; footprint LGA-12_STM -> 74_LIS2DE12TR:LIS2DE12TR
Connections:
- wire segments 45 -> 52
Other:
- moved on the sheet: C4, C5, R27, R28, R29, U12

Commit message: Schematic finished
Parts:
- added R?: PLP-000091, a_pontech:R_0603_1608Metric, symbol 1_pontech:PLP-000091
- R23, R24: DNI (none) -> *DNI
Connections:
- net +3V3: now also R?.1
- net at R23.2, U12.2 (CS): now also R?.2
Other:
- note removed: "MISSING:\n- Add bypass caps (100nf / 10uf)"
Changed lines of the file:
@@
 	1    0    0    -1
 $EndComp
-Text Notes 650  750  0    50   ~ 0
-MISSING:\n- Add bypass caps (100nf / 10uf)
 Text HLabel 4200 2500 1    50   BiDi ~ 0
 I2C-SCL
@@
 	2400 2500 2400 2700
 Wire Wire Line
-	2400 3400 5400 3400
-Wire Wire Line
 	3850 3600 3850 3000
 Wire Wire Line
@@
 $EndComp
 Wire Wire Line
-	4650 3500 5400 3500
-Wire Wire Line
 	3850 3600 5400 3600
 Wire Wire Line
@@
 F 3 "~" H 1600 2850 50  0001 C CNN
 F 4 "0 OHM 0.1W 0603" V 1500 2500 50  0000 L CNN "Info"
-F 5 "*DNI" V 1700 2750 50  0000 C CNN "DNI"
+F 5 "*DNI" V 1600 2850 50  0000 C CNN "DNI"
 	1    1600 2850
 	1    0    0    -1
@@
 F 3 "~" H 1200 2850 50  0001 C CNN
 F 4 "0 OHM 0.1W 0603" V 1100 2500 50  0000 L CNN "Info"
-F 5 "*DNI" V 1300 2750 50  0000 C CNN "DNI"
+F 5 "*DNI" V 1200 2850 50  0000 C CNN "DNI"
 	1    1200 2850
 	1    0    0    -1
@@
 F 3 "~" H 1950 2850 50  0001 C CNN
 F 4 "0 OHM 0.1W 0603" V 1850 2500 50  0000 L CNN "Info"
-F 5 "*DNI" V 2050 2750 50  0000 C CNN "DNI"
+F 5 "*DNI" V 1950 2850 50  0000 C CNN "DNI"
 	1    1950 2850
-	1    0    0    -1
-$EndComp
-$Comp
-L 1_pontech:PLP-000091 R23
-U 1 1 62663ABE
-P 2400 2850
-F 0 "R23" H 2470 2941 50  0000 L CNN
-F 1 "PLP-000091" H 2470 2850 50  0001 L CNN
-F 2 "a_pontech:R_0603_1608Metric" V 2330 2850 50  0001 C CNN
-F 3 "~" H 2400 2850 50  0001 C CNN
-F 4 "0 OHM 0.1W 0603" V 2300 2500 50  0000 L CNN "Info"
-	1    2400 2850
 	1    0    0    -1
 $EndComp
@@
 F 3 "~" H 3500 2850 50  0001 C CNN
 F 4 "0 OHM 0.1W 0603" V 3400 2500 50  0000 L CNN "Info"
+F 5 "*DNI" V 3500 2850 50  0000 C CNN "DNI"
 	1    3500 2850
 	1    0    0    -1
@@
 Wire Wire Line
 	4200 2700 4200 2500
+$Comp
+L 1_pontech:PLP-000091 R?
+U 1 1 6276E5D2
+P 4950 2850
+F 0 "R?" H 5020 2941 50  0000 L CNN
+F 1 "PLP-000091" H 5020 2850 50  0001 L CNN
+F 2 "a_pontech:R_0603_1608Metric" V 4880 2850 50  0001 C CNN
+F 3 "~" H 4950 2850 50  0001 C CNN
+F 4 "0 OHM 0.1W 0603" V 4850 2500 50  0000 L CNN "Info"
+	1    4950 2850
+	1    0    0    -1
+$EndComp
+$Comp
+L 74_Jacob:+3.3V #PWR?
+U 1 1 6276EE33
+P 4950 2500
+F 0 "#PWR?" H 4950 2350 50  0001 C CNN
+F 1 "+3.3V" H 4950 2673 50  0000 C CNN
+F 2 "" H 4950 2500 50  0001 C CNN
+F 3 "" H 4950 2500 50  0001 C CNN
+	1    4950 2500
+	1    0    0    -1
+$EndComp
+Wire Wire Line
+	4950 2500 4950 2700
+Wire Wire Line
+	4650 3500 5400 3500
+Wire Wire Line
+	4950 3000 4950 3400
+Wire Wire Line
+	2400 3400 4950 3400
+Connection ~ 4950 3400
+Wire Wire Line
+	4950 3400 5400 3400
+$Comp
+L 1_pontech:PLP-000091 R23
+U 1 1 62663ABE
+P 2400 2850
+F 0 "R23" H 2470 2941 50  0000 L CNN
+F 1 "PLP-000091" H 2470 2850 50  0001 L CNN
+F 2 "a_pontech:R_0603_1608Metric" V 2330 2850 50  0001 C CNN
+F 3 "~" H 2400 2850 50  0001 C CNN
+F 4 "0 OHM 0.1W 0603" V 2300 2500 50  0000 L CNN "Info"
+F 5 "*DNI" V 2400 2850 50  0000 C CNN "DNI"
+	1    2400 2850
+	1    0    0    -1
+$EndComp
 $EndSCHEMATC

Commit message: Added ESP32 but its going to come off before I am finished.
Parts:
- gave numbers to parts that had none: 1
Changed lines of the file:
@@
 	4200 2700 4200 2500
 $Comp
-L 1_pontech:PLP-000091 R?
+L 1_pontech:PLP-000091 R30
 U 1 1 6276E5D2
 P 4950 2850
-F 0 "R?" H 5020 2941 50  0000 L CNN
+F 0 "R30" H 5020 2941 50  0000 L CNN
 F 1 "PLP-000091" H 5020 2850 50  0001 L CNN
 F 2 "a_pontech:R_0603_1608Metric" V 4880 2850 50  0001 C CNN
@@
 $EndComp
 $Comp
-L 74_Jacob:+3.3V #PWR?
+L 74_Jacob:+3.3V #PWR0135
 U 1 1 6276EE33
 P 4950 2500
-F 0 "#PWR?" H 4950 2350 50  0001 C CNN
+F 0 "#PWR0135" H 4950 2350 50  0001 C CNN
 F 1 "+3.3V" H 4950 2673 50  0000 C CNN
 F 2 "" H 4950 2500 50  0001 C CNN

Commit message: PCB Layout Complete.
Connections:
- net I2C-A0 is gone; now on an unnamed net: R24.1
- net GND: now also R24.2
- net at R22.2, R27.2, U12.3 (SDO/SA0): no longer R24.2
Other:
- moved on the sheet: C4, C5, R24
Changed lines of the file:
@@
 Text HLabel 1600 2500 1    50   Input ~ 0
 SPI-SDI-MOSI
-Text HLabel 3500 2500 1    50   BiDi ~ 0
-I2C-A0
 Wire Wire Line
 	5400 3300 4200 3300
@@
 Wire Wire Line
 	3850 3600 3850 3000
-Wire Wire Line
-	3500 3500 3500 3000
 Wire Wire Line
 	1600 2500 1600 2700
@@
 L 1_pontech:PLP-000068 C4
 U 1 1 6264FAC2
-P 2000 5150
-F 0 "C4" H 2025 5250 50  0000 L CNN
-F 1 "PLP-000068" H 2100 5150 50  0000 L CNN
-F 2 "a_pontech:CAP-NON-POLAR-0603" H 2100 4700 50  0001 L CNN
-F 3 "~" H 2000 5150 50  0001 C CNN
-F 4 "0.1UF 25V 10% X7R 0603" H 2100 5050 50  0000 L CNN "Info"
-	1    2000 5150
+P 2000 5900
+F 0 "C4" H 2025 6000 50  0000 L CNN
+F 1 "PLP-000068" H 2100 5900 50  0000 L CNN
+F 2 "a_pontech:CAP-NON-POLAR-0603" H 2100 5450 50  0001 L CNN
+F 3 "~" H 2000 5900 50  0001 C CNN
+F 4 "0.1UF 25V 10% X7R 0603" H 2100 5800 50  0000 L CNN "Info"
+	1    2000 5900
 	1    0    0    -1
 $EndComp
@@
 L 1_pontech:PLP-000409 C5
 U 1 1 6264FF78
-P 3300 5150
-F 0 "C5" H 3325 5250 50  0000 L CNN
-F 1 "PLP-000409" H 3400 5150 50  0000 L CNN
-F 2 "a_pontech:CAP-NON-POLAR-0603" H 3400 4700 50  0001 L CNN
-F 3 "~" H 3300 5150 50  0001 C CNN
-F 4 "10UF 6.3V 20% X5R 0603" H 3400 5050 50  0000 L CNN "Info"
-	1    3300 5150
-	1    0    0    -1
-$EndComp
-Wire Wire Line
-	3300 5000 3300 4750
-Wire Wire Line
-	2000 5000 2000 4750
-Wire Wire Line
-	2000 5300 2000 5650
+P 3300 5900
+F 0 "C5" H 3325 6000 50  0000 L CNN
+F 1 "PLP-000409" H 3400 5900 50  0000 L CNN
+F 2 "a_pontech:CAP-NON-POLAR-0603" H 3400 5450 50  0001 L CNN
+F 3 "~" H 3300 5900 50  0001 C CNN
+F 4 "10UF 6.3V 20% X5R 0603" H 3400 5800 50  0000 L CNN "Info"
+	1    3300 5900
+	1    0    0    -1
+$EndComp
+Wire Wire Line
+	3300 5750 3300 5500
+Wire Wire Line
+	2000 5750 2000 5500
+Wire Wire Line
+	2000 6050 2000 6400
 $Comp
 L 74_Jacob:+3.3V #PWR0127
 U 1 1 626475ED
-P 2000 4750
-F 0 "#PWR0127" H 2000 4600 50  0001 C CNN
-F 1 "+3.3V" H 2000 4923 50  0000 C CNN
-F 2 "" H 2000 4750 50  0001 C CNN
-F 3 "" H 2000 4750 50  0001 C CNN
-	1    2000 4750
+P 2000 5500
+F 0 "#PWR0127" H 2000 5350 50  0001 C CNN
+F 1 "+3.3V" H 2000 5673 50  0000 C CNN
+F 2 "" H 2000 5500 50  0001 C CNN
+F 3 "" H 2000 5500 50  0001 C CNN
+	1    2000 5500
 	1    0    0    -1
 $EndComp
@@
 L 74_Jacob:+3.3V #PWR0128
 U 1 1 626484B4
-P 3300 4750
-F 0 "#PWR0128" H 3300 4600 50  0001 C CNN
-F 1 "+3.3V" H 3300 4923 50  0000 C CNN
-F 2 "" H 3300 4750 50  0001 C CNN
-F 3 "" H 3300 4750 50  0001 C CNN
-	1    3300 4750
+P 3300 5500
+F 0 "#PWR0128" H 3300 5350 50  0001 C CNN
+F 1 "+3.3V" H 3300 5673 50  0000 C CNN
+F 2 "" H 3300 5500 50  0001 C CNN
+F 3 "" H 3300 5500 50  0001 C CNN
+	1    3300 5500
 	1    0    0    -1
 $EndComp
@@
 L 74_Jacob:GND #PWR0131
 U 1 1 626496EF
-P 2000 5650
-F 0 "#PWR0131" H 2000 5400 50  0001 C CNN
-F 1 "GND" H 2000 5477 50  0000 C CNN
-F 2 "" H 2000 5650 50  0001 C CNN
-F 3 "" H 2000 5650 50  0001 C CNN
-	1    2000 5650
-	1    0    0    -1
-$EndComp
-Wire Wire Line
-	3300 5300 3300 5650
+P 2000 6400
+F 0 "#PWR0131" H 2000 6150 50  0001 C CNN
+F 1 "GND" H 2000 6227 50  0000 C CNN
+F 2 "" H 2000 6400 50  0001 C CNN
+F 3 "" H 2000 6400 50  0001 C CNN
+	1    2000 6400
+	1    0    0    -1
+$EndComp
+Wire Wire Line
+	3300 6050 3300 6400
 $Comp
 L 74_Jacob:GND #PWR0132
 U 1 1 6264A815
-P 3300 5650
-F 0 "#PWR0132" H 3300 5400 50  0001 C CNN
-F 1 "GND" H 3300 5477 50  0000 C CNN
-F 2 "" H 3300 5650 50  0001 C CNN
-F 3 "" H 3300 5650 50  0001 C CNN
-	1    3300 5650
+P 3300 6400
+F 0 "#PWR0132" H 3300 6150 50  0001 C CNN
+F 1 "GND" H 3300 6227 50  0000 C CNN
+F 2 "" H 3300 6400 50  0001 C CNN
+F 3 "" H 3300 6400 50  0001 C CNN
+	1    3300 6400
 	1    0    0    -1
 $EndComp
@@
 L 1_pontech:PLP-000091 R24
 U 1 1 62663FDF
-P 3500 2850
-F 0 "R24" H 3570 2941 50  0000 L CNN
-F 1 "PLP-000091" H 3570 2850 50  0001 L CNN
-F 2 "a_pontech:R_0603_1608Metric" V 3430 2850 50  0001 C CNN
-F 3 "~" H 3500 2850 50  0001 C CNN
-F 4 "0 OHM 0.1W 0603" V 3400 2500 50  0000 L CNN "Info"
-F 5 "*DNI" V 3500 2850 50  0000 C CNN "DNI"
-	1    3500 2850
-	1    0    0    -1
-$EndComp
-Wire Wire Line
-	3500 2700 3500 2500
+P 3500 4000
+F 0 "R24" H 3570 4091 50  0000 L CNN
+F 1 "PLP-000091" H 3570 4000 50  0001 L CNN
+F 2 "a_pontech:R_0603_1608Metric" V 3430 4000 50  0001 C CNN
+F 3 "~" H 3500 4000 50  0001 C CNN
+F 4 "0 OHM 0.1W 0603" V 3400 3650 50  0000 L CNN "Info"
+F 5 "*DNI" V 3500 4000 50  0000 C CNN "DNI"
+	1    3500 4000
+	1    0    0    -1
+$EndComp
 $Comp
 L 1_pontech:PLP-000091 R25
@@
 	1    0    0    -1
 $EndComp
+$Comp
+L 74_Jacob:GND #PWR?
+U 1 1 6277FCB9
+P 3500 4450
+F 0 "#PWR?" H 3500 4200 50  0001 C CNN
+F 1 "GND" H 3500 4277 50  0000 C CNN
+F 2 "" H 3500 4450 50  0001 C CNN
+F 3 "" H 3500 4450 50  0001 C CNN
+	1    3500 4450
+	1    0    0    -1
+$EndComp
+Wire Wire Line
+	3500 4150 3500 4450
+Wire Wire Line
+	3500 3850 3500 3500
 $EndSCHEMATC
