File: KiCAD/ClassProject/Spring2022/Spring2022.kicad_pcb (KiCad board)
At the start: 2 copper layers, 211 x 39 mm, 64 parts, among them U1 FUB-MINI, U10 LM35-LP, U11 SHT40-AD1B-R3, U12 LGA-12_STM, U2 74HC595, U3 74HC595, U4 74HC595, U5 74HC595, U6 74HC595, U7 74HC595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

Commit message: Revert "Upgraded to KiCAD 6.0"
This reverts commit 6b4ca58081787079494b2a2522a3e7ee5416242f.
Connections:
- net ~{CS-ACC} renamed ~CS-ACC
- net ~{INT1-ACC} renamed ~INT1-ACC
- net ~{INT2-ACC} renamed ~INT2-ACC
- net ~{LED-OE} renamed ~LED-OE
Other:
- net class Default added: clearance 0.127, trace_width 0.127, via_dia 0.8, via_drill 0.4
